File: hw/board1/scehmatic1.brd (EAGLE design)
At the start: 100 x 80 mm, 8 parts, among them IC1 LM317MBSTT3

Commit message: deleted component from schematic and thus board
Parts:
- removed IC1: LM317MBSTT3, v-reg:SOT223
Connections:
- net N$1: no longer IC1.1
- net VIN: no longer IC1.3
- net VO: no longer IC1.4
Changed lines of the file:
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@@
 <element name="D1" library="diode" package="DO41-10" package3d_urn="urn:adsk.eagle:package:43336/1" value="1N4002" x="-19.05" y="21.59"/>
 <element name="D2" library="diode" package="DO41-10" package3d_urn="urn:adsk.eagle:package:43336/1" value="1N4002" x="-31.75" y="21.59"/>
-<element name="IC1" library="v-reg" library_urn="urn:adsk.eagle:library:409" package="SOT223" package3d_urn="urn:adsk.eagle:package:30370/1" value="LM317MBSTT3" x="-24.13" y="13.97">
-<attribute name="PARTNUMBER" value="LM317" x="-24.13" y="13.97" size="1.778" layer="27" display="off"/>
-</element>
 <element name="R1" library="resistor" library_urn="urn:adsk.eagle:library:348" package="M0805" package3d_urn="urn:adsk.eagle:package:26079/1" value="240Ω" x="-16.51" y="29.21"/>
 <element name="R2" library="resistor" library_urn="urn:adsk.eagle:library:348" package="M0805" package3d_urn="urn:adsk.eagle:package:26079/1" value="4.4K" x="-21.59" y="29.21"/>
@@
 <contactref element="R1" pad="1"/>
 <contactref element="C3" pad="+"/>
-<contactref element="IC1" pad="1"/>
 <contactref element="R2" pad="2"/>
-<wire x1="-26.43" y1="10.82" x2="-27.23" y2="5.08" width="0" layer="19" extent="1-1"/>
-<wire x1="-26.67" y1="21.59" x2="-26.43" y2="10.82" width="0" layer="19" extent="1-1"/>
+<wire x1="-26.67" y1="21.59" x2="-27.23" y2="5.08" width="0" layer="19" extent="1-1"/>
 <wire x1="-20.64" y1="29.21" x2="-26.67" y2="21.59" width="0" layer="19" extent="1-1"/>
 <wire x1="-17.46" y1="29.21" x2="-20.64" y2="29.21" width="0" layer="19" extent="1-1"/>
@@
 <signal name="VO">
 <contactref element="D2" pad="C"/>
-<contactref element="IC1" pad="4"/>
 <contactref element="R1" pad="2"/>
 <contactref element="D1" pad="A"/>
 <contactref element="C2" pad="+"/>
-<wire x1="-24.13" y1="17.12" x2="-36.83" y2="21.59" width="0" layer="19" extent="1-1"/>
-<wire x1="-13.97" y1="21.59" x2="-24.13" y2="17.12" width="0" layer="19" extent="1-1"/>
-<wire x1="-15.56" y1="29.21" x2="-13.97" y2="21.59" width="0" layer="19" extent="1-1"/>
-<wire x1="-15.8" y1="5.08" x2="-24.13" y2="17.12" width="0" layer="19" extent="1-1"/>
+<wire x1="-15.56" y1="29.21" x2="-36.83" y2="21.59" width="0" layer="19" extent="1-1"/>
+<wire x1="-13.97" y1="21.59" x2="-15.56" y2="29.21" width="0" layer="19" extent="1-1"/>
+<wire x1="-15.8" y1="5.08" x2="-13.97" y2="21.59" width="0" layer="19" extent="1-1"/>
 </signal>
 <signal name="VIN">
 <contactref element="C1" pad="1"/>
-<contactref element="IC1" pad="3"/>
 <contactref element="D1" pad="C"/>
-<wire x1="-21.83" y1="10.82" x2="-36.83" y2="12.7" width="0" layer="19" extent="1-1"/>
-<wire x1="-24.13" y1="21.59" x2="-21.83" y2="10.82" width="0" layer="19" extent="1-1"/>
+<wire x1="-24.13" y1="21.59" x2="-36.83" y2="12.7" width="0" layer="19" extent="1-1"/>
 </signal>
 <signal name="N$2">
